File: mosfet_brd.brd (EAGLE design)
At the start: 60 x 50 mm, 10 parts, among them Q1 IRF2807, T1 BC547

Commit message: Pasta reorganizada
Parts:
- removed OUTPUT: (no value), con-ptr500:AK300/2
- added OUTPUT1, OUTPUT2: (no value), con-ptr500:AK300/2
- moved LED1 6.08 mm to (35.0, 39.0)
- moved T1 2.00 mm to (22.0, 38.0), turned to 180 degrees
Connections:
- net GND: now also OUTPUT2.2
- net GND-O: now also OUTPUT1.2; no longer OUTPUT.2
- net VCC: now also OUTPUT1.1, OUTPUT2.1; no longer OUTPUT.1
Routing:
- net GND: track 86.7 -> 156.7 mm
- net GND-O: track 69.5 -> 51.1 mm
- net VCC: track 120.5 -> 112.2 mm
- net N$2: track 14.2 -> 8.69 mm
- net N$5: track 64.2 -> 59.3 mm
- net N$7: track 22.0 -> 24.7 mm

Commit message: Peq mudanças
Parts:
- moved T1 4.90 mm to (17.2, 37.0)
Routing:
- net GND: track 156.7 -> 153.6 mm
- net N$2: track 8.69 -> 5.77 mm
- net N$5: track 59.3 -> 56.8 mm
- net GND-O: track 51.1 -> 52.2 mm
